File: connector.kicad_pcb (KiCad board)
At the start: 2 copper layers, 22.2 x 17.8 mm, 13 parts, among them P1 CONN_01X08, P2 CONN_01X01, P3 CONN_01X01

Commit message: Connector
Parts:
- moved P2 12.7 mm to (185.4, 119.4)
- moved P3 12.7 mm to (185.4, 106.7)
- moved P1 5.97 mm to (174.2, 113.0), turned to 270 degrees
Routing:
- net GND: track 29.6 -> 45.4 mm, vias 3 -> 8
- net Net-(P1-Pad2): track 23.5 -> 12.7 mm, vias 1 -> 0
- net Net-(P1-Pad3): track 20.8 -> 13.4 mm
- net +5V: track 41.0 -> 35.9 mm, vias 3 -> 2
- net Net-(P1-Pad7): track 16.4 -> 21.1 mm, vias 0 -> 1
- net Net-(P1-Pad6): track 15.7 -> 14.3 mm, vias 0 -> 1
