File: moto-dcdc.kicad_pcb (KiCad board)
At the start: 2 copper layers, 42.7 x 44.6 mm, 21 parts, among them P1 CONN_01X01, P2 CONN_01X01, P3 CONN_01X01, P4 CONN_01X01, P5 CONN_01X01, U1 LMR14050

Commit message: Gerbers
Routing:
- net GND: vias 158 -> 170
Changed lines of the file:
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@@
-(kicad_pcb (version 4) (host pcbnew 0.201604071231+6672~43~ubuntu15.10.1-product)
+(kicad_pcb (version 4) (host pcbnew 4.1.0-alpha+201606301453+6958~45~ubuntu15.10.1-product)
   (general
     (links 34)
     (no_connects 0)
-    (area 125.822727 76.160766 168.608846 120.862352)
+    (area 125.476 68.274167 181.990001 131.269001)
     (thickness 1.6)
-    (drawings 266)
-    (tracks 562)
+    (drawings 268)
+    (tracks 574)
     (zones 0)
     (modules 21)
@@
   )
   (setup
-    (last_trace_width 0.8128)
+    (last_trace_width 0.25)
     (user_trace_width 0.4064)
     (user_trace_width 0.8128)
@@
     (pad_to_mask_clearance 0.2)
     (aux_axis_origin 0 0)
-    (visible_elements FFFFEF7F)
+    (visible_elements FFFFFF7F)
     (pcbplotparams
-      (layerselection 0x00030_ffffffff)
+      (layerselection 0x010f0_ffffffff)
       (usegerberextensions false)
+      (usegerberattributes true)
       (excludeedgelayer true)
       (linewidth 0.100000)
@@
       (psnegative false)
       (psa4output false)
-      (plotreference true)
+      (plotreference false)
       (plotvalue true)
       (plotinvisibletext false)
       (padsonsilk false)
-      (subtractmaskfromsilk false)
+      (subtractmaskfromsilk true)
       (outputformat 1)
       (mirror false)
-      (drillshape 1)
+      (drillshape 0)
       (scaleselection 1)
-      (outputdirectory ""))
+      (outputdirectory gerbers/moto-dcdc/))
   )
   (net 0 "")
@@
   (module iwasz:HSOIC_8_powerpad (layer F.Cu)
     (at 148.844 115.062 270)
-    (fp_text reference U1 (at 3.2 1.6 360) (layer F.SilkS)
+    (fp_text reference U1 (at 3.2 1.6) (layer F.SilkS)
       (effects (font (size 1 1) (thickness 0.15)))
     )
@@
     (at 156.972 105.918 270)
     (descr "<b>DPAK</b> CASE 369-07<br>\nSource MOTOROLA / ON Semiconductor mjd32-d.pdf")
-    (fp_text reference D3 (at -3.81 2.94 360) (layer F.SilkS)
+    (fp_text reference D3 (at -3.81 2.94) (layer F.SilkS)
       (effects (font (size 1 1) (thickness 0.15)) (justify left bottom))
     )
-    (fp_text value MBRD835LT4G (at 5.08 2.94 360) (layer F.SilkS)
+    (fp_text value MBRD835LT4G (at 5.08 2.94) (layer F.SilkS)
       (effects (font (size 1 1) (thickness 0.15)) (justify left bottom))
     )
@@
     (pad 1 thru_hole circle (at 0 0) (size 2.54 2.54) (drill 1.3208) (layers *.Cu *.Mask)
       (net 1 GND))
+  )
+  (dimension 42.926 (width 0.3) (layer Dwgs.User)
+    (gr_text "42,926 mm" (at 147.193 129.874) (layer Dwgs.User)
+      (effects (font (size 1.5 1.5) (thickness 0.3)))
+    )
+    (feature1 (pts (xy 168.656 110.236) (xy 168.656 131.224)))
+    (feature2 (pts (xy 125.73 110.236) (xy 125.73 131.224)))
+    (crossbar (pts (xy 125.73 128.524) (xy 168.656 128.524)))
+    (arrow1a (pts (xy 168.656 128.524) (xy 167.529496 129.110421)))
+    (arrow1b (pts (xy 168.656 128.524) (xy 167.529496 127.937579)))
+    (arrow2a (pts (xy 125.73 128.524) (xy 126.856504 129.110421)))
+    (arrow2b (pts (xy 125.73 128.524) (xy 126.856504 127.937579)))
+  )
+  (dimension 44.704 (width 0.3) (layer Dwgs.User)
+    (gr_text "44,704 mm" (at 175.34 98.552 270) (layer Dwgs.User)
+      (effects (font (size 1.5 1.5) (thickness 0.3)))
+    )
+    (feature1 (pts (xy 157.988 120.904) (xy 176.69 120.904)))
+    (feature2 (pts (xy 157.988 76.2) (xy 176.69 76.2)))
+    (crossbar (pts (xy 173.99 76.2) (xy 173.99 120.904)))
+    (arrow1a (pts (xy 173.99 120.904) (xy 173.403579 119.777496)))
+    (arrow1b (pts (xy 173.99 120.904) (xy 174.576421 119.777496)))
+    (arrow2a (pts (xy 173.99 76.2) (xy 173.403579 77.326504)))
+    (arrow2b (pts (xy 173.99 76.2) (xy 174.576421 77.326504)))
   )
   (gr_text GND (at 150.114 79.248) (layer F.SilkS)
@@
   (gr_line (start 162.675561 83.280174) (end 162.353094 83.027066) (layer Edge.Cuts) (width 0.1))
   (gr_line (start 148.336 107.696) (end 148.114492 107.878762) (layer Edge.Cuts) (width 0.1))
+  (via (at 147.828 116.332) (size 0.6) (drill 0.4) (layers F.Cu B.Cu) (net 1))
+  (via (at 147.066 116.332) (size 0.6) (drill 0.4) (layers F.Cu B.Cu) (net 1))
+  (via (at 146.304 116.332) (size 0.6) (drill 0.4) (layers F.Cu B.Cu) (net 1))
+  (via (at 146.304 115.57) (size 0.6) (drill 0.4) (layers F.Cu B.Cu) (net 1))
+  (via (at 147.066 115.57) (size 0.6) (drill 0.4) (layers F.Cu B.Cu) (net 1))
+  (via (at 147.828 115.57) (size 0.6) (drill 0.4) (layers F.Cu B.Cu) (net 1))
+  (via (at 147.828 114.808) (size 0.6) (drill 0.4) (layers F.Cu B.Cu) (net 1))
+  (via (at 147.066 114.808) (size 0.6) (drill 0.4) (layers F.Cu B.Cu) (net 1))
+  (via (at 146.304 114.808) (size 0.6) (drill 0.4) (layers F.Cu B.Cu) (net 1))
+  (via (at 147.828 114.046) (size 0.6) (drill 0.4) (layers F.Cu B.Cu) (net 1))
+  (via (at 147.066 114.046) (size 0.6) (drill 0.4) (layers F.Cu B.Cu) (net 1))
+  (via (at 146.304 114.046) (size 0.6) (drill 0.4) (layers F.Cu B.Cu) (net 1))
   (segment (start 155.956 93.726) (end 153.797 91.567) (width 0.4064) (layer F.Cu) (net 1))
   (segment (start 153.797 91.567) (end 151.511 91.567) (width 0.4064) (layer F.Cu) (net 1))
